File: heater.sch (EAGLE design)
At the start: 15 parts

Commit message: Add files via upload
Parts:
- R1: value 5.1k -> 100
- R2: value 100 -> 5.1k
- VT1: value IRF9540 -> 2N2222; device transistor-fet:IRF9530 -> transistor:2N2222
- VT4: value 2N2222 -> IRF9540; device transistor:2N2222 -> transistor-fet:IRF9530
- renumbered R19 to R4, R9 to R20
Connections:
- net +24V: now also R2.2, VT4.S; no longer R1.2, VT1.S
- net N$3: now also VT4.D; no longer VT1.D
- net N$4: now also R3.1, VT4.G; no longer R2.1, VT1.G
- net N$5: now also R3.2; no longer R2.2
- net N$6: now also R2.1, VT1.C; no longer R1.1, VT4.C
- net N$7: now also VT1.E; no longer VT4.E
- net N$8: now also R1.1, VT1.B; no longer R3.1, VT4.B
- net N$9: now also R1.2; no longer R3.2
Other:
- moved on the sheet: R1, R2, R3, VT1, VT4
Changed lines of the file:
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@@
 <part name="L1" library="inductor-neosid" library_urn="urn:adsk.eagle:library:241" deviceset="SD8" device="" package3d_urn="urn:adsk.eagle:package:14649/1" value="50-100uH"/>
 <part name="VD2" library="diode" library_urn="urn:adsk.eagle:library:210" deviceset="1N4004" device="" package3d_urn="urn:adsk.eagle:package:43336/1" value="FR107"/>
-<part name="R1" library="rcl" library_urn="urn:adsk.eagle:library:334" deviceset="R-EU_" device="0207/10" package3d_urn="urn:adsk.eagle:package:23491/1" value="5.1k"/>
-<part name="VT1" library="transistor-fet" library_urn="urn:adsk.eagle:library:396" deviceset="IRF9530" device="" package3d_urn="urn:adsk.eagle:package:28520/1" value="IRF9540"/>
+<part name="R2" library="rcl" library_urn="urn:adsk.eagle:library:334" deviceset="R-EU_" device="0207/10" package3d_urn="urn:adsk.eagle:package:23491/1" value="5.1k"/>
+<part name="VT4" library="transistor-fet" library_urn="urn:adsk.eagle:library:396" deviceset="IRF9530" device="" package3d_urn="urn:adsk.eagle:package:28520/1" value="IRF9540"/>
 <part name="VD1" library="diode" library_urn="urn:adsk.eagle:library:210" deviceset="ZENER-DIODE" device="C1702-15" package3d_urn="urn:adsk.eagle:package:43351/1" value="18v"/>
 <part name="VT2" library="transistor" library_urn="urn:adsk.eagle:library:402" deviceset="2N2222" device="" package3d_urn="urn:adsk.eagle:package:29892/2"/>
 <part name="VT3" library="transistor" library_urn="urn:adsk.eagle:library:402" deviceset="*-PNP-" device="TO18-EBC" package3d_urn="urn:adsk.eagle:package:29892/2" technology="2N2907" value="2N2907"/>
-<part name="R2" library="rcl" library_urn="urn:adsk.eagle:library:334" deviceset="R-EU_" device="0207/10" package3d_urn="urn:adsk.eagle:package:23491/1" value="100"/>
 <part name="R3" library="rcl" library_urn="urn:adsk.eagle:library:334" deviceset="R-EU_" device="0207/10" package3d_urn="urn:adsk.eagle:package:23491/1" value="100"/>
+<part name="R1" library="rcl" library_urn="urn:adsk.eagle:library:334" deviceset="R-EU_" device="0207/10" package3d_urn="urn:adsk.eagle:package:23491/1" value="100"/>
 <part name="R5" library="rcl" library_urn="urn:adsk.eagle:library:334" deviceset="R-EU_" device="0207/10" package3d_urn="urn:adsk.eagle:package:23491/1" value="1k"/>
-<part name="R9" library="rcl" library_urn="urn:adsk.eagle:library:334" deviceset="R-EU_" device="0207/10" package3d_urn="urn:adsk.eagle:package:23491/1" value="0.11, 2W"/>
+<part name="R20" library="rcl" library_urn="urn:adsk.eagle:library:334" deviceset="R-EU_" device="0207/10" package3d_urn="urn:adsk.eagle:package:23491/1" value="0.11, 2W"/>
 <part name="P+1" library="supply1" library_urn="urn:adsk.eagle:library:371" deviceset="+24V" device=""/>
 <part name="GND1" library="supply1" library_urn="urn:adsk.eagle:library:371" deviceset="GND" device=""/>
-<part name="VT4" library="transistor" library_urn="urn:adsk.eagle:library:402" deviceset="2N2222" device="" package3d_urn="urn:adsk.eagle:package:29892/2"/>
+<part name="VT1" library="transistor" library_urn="urn:adsk.eagle:library:402" deviceset="2N2222" device="" package3d_urn="urn:adsk.eagle:package:29892/2"/>
 <part name="PA0,PWM" library="pinhead" library_urn="urn:adsk.eagle:library:325" deviceset="PINHD-1X1" device="" package3d_urn="urn:adsk.eagle:package:22485/2"/>
-<part name="R19" library="rcl" library_urn="urn:adsk.eagle:library:334" deviceset="R-EU_" device="0207/10" package3d_urn="urn:adsk.eagle:package:23491/1" value="100k"/>
+<part name="R4" library="rcl" library_urn="urn:adsk.eagle:library:334" deviceset="R-EU_" device="0207/10" package3d_urn="urn:adsk.eagle:package:23491/1" value="100k"/>
 </parts>
 <sheets>
@@
 <attribute name="VALUE" x="-5.3086" y="35.56" size="1.778" layer="96" rot="R90"/>
 </instance>
-<instance part="R1" gate="G$1" x="27.94" y="93.98" rot="R90">
+<instance part="R2" gate="G$1" x="27.94" y="93.98" rot="R90">
 <attribute name="NAME" x="26.4414" y="90.17" size="1.778" layer="95" rot="R90"/>
 <attribute name="VALUE" x="31.242" y="90.17" size="1.778" layer="96" rot="R90"/>
 </instance>
-<instance part="VT1" gate="G$1" x="-12.7" y="71.12" rot="R180">
+<instance part="VT4" gate="G$1" x="-12.7" y="71.12" rot="R180">
 <attribute name="VALUE" x="-1.27" y="71.12" size="1.778" layer="96" rot="R180"/>
 <attribute name="NAME" x="-3.81" y="68.58" size="1.778" layer="95" rot="R180"/>
@@
 <attribute name="VALUE" x="22.86" y="58.42" size="1.778" layer="96" rot="MR0"/>
 </instance>
-<instance part="R2" gate="G$1" x="5.08" y="73.66">
+<instance part="R3" gate="G$1" x="5.08" y="73.66">
 <attribute name="NAME" x="1.27" y="75.1586" size="1.778" layer="95"/>
 <attribute name="VALUE" x="1.27" y="70.358" size="1.778" layer="96"/>
 </instance>
-<instance part="R3" gate="G$1" x="45.72" y="50.8">
+<instance part="R1" gate="G$1" x="45.72" y="50.8">
 <attribute name="NAME" x="41.91" y="52.2986" size="1.778" layer="95"/>
 <attribute name="VALUE" x="41.91" y="47.498" size="1.778" layer="96"/>
@@
 <attribute name="VALUE" x="31.242" y="31.75" size="1.778" layer="96" rot="R90"/>
 </instance>
-<instance part="R9" gate="G$1" x="-17.78" y="33.02" rot="R90">
+<instance part="R20" gate="G$1" x="-17.78" y="33.02" rot="R90">
 <attribute name="NAME" x="-19.2786" y="29.21" size="1.778" layer="95" rot="R90"/>
 <attribute name="VALUE" x="-14.478" y="29.21" size="1.778" layer="96" rot="R90"/>
@@
 <attribute name="VALUE" x="-20.32" y="17.78" size="1.778" layer="96"/>
 </instance>
-<instance part="VT4" gate="G$1" x="30.48" y="50.8" rot="MR0">
+<instance part="VT1" gate="G$1" x="30.48" y="50.8" rot="MR0">
 <attribute name="NAME" x="33.02" y="55.88" size="1.778" layer="95" rot="MR0"/>
 <attribute name="VALUE" x="38.1" y="45.72" size="1.778" layer="96" rot="MR0"/>
@@
 <attribute name="VALUE" x="54.61" y="45.72" size="1.778" layer="96"/>
 </instance>
-<instance part="R19" gate="G$1" x="0" y="91.44" rot="R90">
+<instance part="R4" gate="G$1" x="0" y="91.44" rot="R90">
 <attribute name="NAME" x="-1.4986" y="87.63" size="1.778" layer="95" rot="R90"/>
 <attribute name="VALUE" x="3.302" y="87.63" size="1.778" layer="96" rot="R90"/>
@@
 <segment>
 <pinref part="JP1" gate="G$1" pin="1"/>
-<pinref part="R9" gate="G$1" pin="2"/>
+<pinref part="R20" gate="G$1" pin="2"/>
 <wire x1="-27.94" y1="43.18" x2="-17.78" y2="43.18" width="0.1524" layer="91"/>
 <wire x1="-17.78" y1="43.18" x2="-17.78" y2="38.1" width="0.1524" layer="91"/>
@@
 <segment>
 <pinref part="GND1" gate="1" pin="GND"/>
-<pinref part="R9" gate="G$1" pin="1"/>
+<pinref part="R20" gate="G$1" pin="1"/>
 <wire x1="-17.78" y1="22.86" x2="-17.78" y2="25.4" width="0.1524" layer="91"/>
 <wire x1="-17.78" y1="25.4" x2="-17.78" y2="27.94" width="0.1524" layer="91"/>
@@
 <pinref part="L1" gate="G$1" pin="2"/>
 <wire x1="-17.78" y1="60.96" x2="-17.78" y2="58.42" width="0.1524" layer="91"/>
-<pinref part="VT1" gate="G$1" pin="D"/>
+<pinref part="VT4" gate="G$1" pin="D"/>
 <wire x1="-17.78" y1="60.96" x2="-17.78" y2="68.58" width="0.1524" layer="91"/>
 <junction x="-17.78" y="60.96"/>
@@
 <net name="+24V" class="0">
 <segment>
-<pinref part="VT1" gate="G$1" pin="S"/>
+<pinref part="VT4" gate="G$1" pin="S"/>
 <pinref part="P+1" gate="1" pin="+24V"/>
 <wire x1="-17.78" y1="73.66" x2="-17.78" y2="101.6" width="0.1524" layer="91"/>
 <wire x1="-17.78" y1="101.6" x2="-17.78" y2="106.68" width="0.1524" layer="91"/>
-<pinref part="R1" gate="G$1" pin="2"/>
+<pinref part="R2" gate="G$1" pin="2"/>
 <wire x1="27.94" y1="99.06" x2="27.94" y2="101.6" width="0.1524" layer="91"/>
 <wire x1="27.94" y1="101.6" x2="12.7" y2="101.6" width="0.1524" layer="91"/>
@@
 <wire x1="-7.62" y1="101.6" x2="-7.62" y2="86.36" width="0.1524" layer="91"/>
 <junction x="-7.62" y="101.6"/>
-<pinref part="R19" gate="G$1" pin="2"/>
+<pinref part="R4" gate="G$1" pin="2"/>
 <wire x1="0" y1="96.52" x2="0" y2="101.6" width="0.1524" layer="91"/>
 <junction x="0" y="101.6"/>
@@
 <net name="N$4" class="0">
 <segment>
-<pinref part="VT1" gate="G$1" pin="G"/>
+<pinref part="VT4" gate="G$1" pin="G"/>
 <pinref part="VD1" gate="G$1" pin="A"/>
 <wire x1="-7.62" y1="73.66" x2="-7.62" y2="81.28" width="0.1524" layer="91"/>
-<pinref part="R2" gate="G$1" pin="1"/>
+<pinref part="R3" gate="G$1" pin="1"/>
 <wire x1="-7.62" y1="73.66" x2="0" y2="73.66" width="0.1524" layer="91"/>
 <junction x="-7.62" y="73.66"/>
-<pinref part="R19" gate="G$1" pin="1"/>
+<pinref part="R4" gate="G$1" pin="1"/>
 <wire x1="0" y1="86.36" x2="0" y2="73.66" width="0.1524" layer="91"/>
 <junction x="0" y="73.66"/>
@@
 <net name="N$5" class="0">
 <segment>
-<pinref part="R2" gate="G$1" pin="2"/>
+<pinref part="R3" gate="G$1" pin="2"/>
 <wire x1="10.16" y1="73.66" x2="12.7" y2="73.66" width="0.1524" layer="91"/>
 <pinref part="VT2" gate="G$1" pin="E"/>
@@
 <pinref part="VT3" gate="G$1" pin="B"/>
 <wire x1="27.94" y1="63.5" x2="17.78" y2="63.5" width="0.1524" layer="91"/>
-<pinref part="R1" gate="G$1" pin="1"/>
+<pinref part="R2" gate="G$1" pin="1"/>
 <wire x1="27.94" y1="83.82" x2="27.94" y2="88.9" width="0.1524" layer="91"/>
 <junction x="27.94" y="83.82"/>
-<pinref part="VT4" gate="G$1" pin="C"/>
+<pinref part="VT1" gate="G$1" pin="C"/>
 <wire x1="27.94" y1="55.88" x2="27.94" y2="63.5" width="0.1524" layer="91"/>
 <junction x="27.94" y="63.5"/>
@@
 <net name="N$7" class="0">
 <segment>
-<pinref part="VT4" gate="G$1" pin="E"/>
+<pinref part="VT1" gate="G$1" pin="E"/>
 <pinref part="R5" gate="G$1" pin="2"/>
 <wire x1="27.94" y1="45.72" x2="27.94" y2="40.64" width="0.1524" layer="91"/>
@@
 <net name="N$8" class="0">
 <segment>
-<pinref part="R3" gate="G$1" pin="1"/>
-<pinref part="VT4" gate="G$1" pin="B"/>
+<pinref part="R1" gate="G$1" pin="1"/>
+<pinref part="VT1" gate="G$1" pin="B"/>
 <wire x1="40.64" y1="50.8" x2="33.02" y2="50.8" width="0.1524" layer="91"/>
 </segment>
@@
 <net name="N$9" class="0">
 <segment>
-<pinref part="R3" gate="G$1" pin="2"/>
+<pinref part="R1" gate="G$1" pin="2"/>
 <pinref part="PA0,PWM" gate="G$1" pin="1"/>
 <wire x1="50.8" y1="50.8" x2="58.42" y2="50.8" width="0.1524" layer="91"/>
