File: stm32_hakko.sch (EAGLE design)
At the start: 41 parts, among them U1 AT24C32A

Commit message: Add files via upload
Parts:
- C1: value 1uF -> 100n
- C5: value 100n -> 1uF
- R1: value 5.1k -> 100
- R11: value 500k -> 10k; device pot:TRIM_EU-RJ9W -> rcl:R-EU_0204/5
- R12: value 50k -> 0.11, 2W
- R13: value 470 -> 2k
- R14: value 1k -> 2k
- R15: value 2k -> THERMISTOR; device rcl:R-EU_0204/5 -> varistor:THERMISTOR-2,5
- R16: value 2k -> 470
- R17: value THERMISTOR -> 100k; device varistor:THERMISTOR-2,5 -> rcl:R-EU_0204/5
- R18: value 10k -> 1k
- R19, R6: value 100k -> 10k
- R2: value 100 -> 5.1k
- R4: value 10k -> 100k
- R8: value 10k -> 500k; device rcl:R-EU_0204/5 -> pot:TRIM_EU-RJ9W
- R9: value 0.11, 2W -> 50k
- VT1: value IRF9540 -> 2N2222; device transistor-fet:IRF9530 -> transistor:2N2222
- VT4: value 2N2222 -> IRF9540; device transistor:2N2222 -> transistor-fet:IRF9530
- renumbered D2 to D1, VD3 to VD2
Connections:
- net +24V: now also R2.2, R4.2, VT4.S; no longer R1.2, R19.2, VT1.S
- net +3V3: now also R13.2, R14.2, R6.2; no longer R15.2, R16.2, R18.2
- net GND: now also C1.1, C2.1, C4.2, C5.2, R12.1, R15.1, R18.1; no longer C1.2, C2.2, C4.1, C5.1, R10.1, R17.1, R9.1
- net N$1: now also R14.1; no longer R15.1
- net N$10: now also C2.2; no longer C4.2
- net N$11: now also C1.2; no longer C3.2
- net N$12: now also R8.E, R9.1; no longer R11.E, R12.1
- net N$13: now also R7.1; no longer R13.1
- net N$14: now also R10.2, R9.2; no longer R12.2, R14.2
- net N$15: now also R11.1; no longer R4.1
- net N$16: now also R11.2, R12.2, R19.2; no longer R4.2, R8.2, R9.2
- net N$17: now also VT4.D; no longer VT1.D
- net N$18: now also C4.1, R16.1, R17.1; no longer C2.1, R6.1, R7.1
- net N$19: now also R17.2, R18.2; no longer R10.2, R6.2
- net N$2: now also R13.1; no longer R16.1
- net N$20: now also R7.2, R8.A, R8.S; no longer R11.A, R11.S, R13.2
- net N$21: now also R16.2; no longer R7.2
- net N$22: now also C5.1, R19.1; no longer C1.1, R8.1
- net N$23: now also R3.2, R4.1, VT4.G; no longer R19.1, R2.2, VT1.G
- net N$24: now also R3.1; no longer R2.1
- net N$25: now also R2.1, VT1.C; no longer R1.1, VT4.C
- net N$26: now also VT1.E; no longer VT4.E
- net N$27: now also R1.2, VT1.B; no longer R3.2, VT4.B
- net N$28: now also R1.1; no longer R3.1
- net N$29: now also R15.2, R6.1; no longer R17.2, R18.1
- net N$9: now also C3.2; no longer C5.2
- net VD3: now also R10.1; no longer R14.1
Other:
- moved on the sheet: C1, C2, C3, C4, C5, R1, R10, R12, R13, R14, R16, R18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
