File: eagle/F1-T12_heater.sch (EAGLE design)
At the start: 9 parts

Commit message: Add files via upload
Connections:
- removed net N$16: D1.C, IRON.1, IRON.2, R10.2, VT2.D
- new net V+: D1.C, IRON.1, VT2.D
- new net V-: IRON.2, R10.2
Changed lines of the file:
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@@
 <?xml version="1.0" encoding="utf-8"?>
 <!DOCTYPE eagle SYSTEM "eagle.dtd">
-<eagle version="9.2.0">
+<eagle version="9.6.1">
 <drawing>
 <settings>
@@
 <part name="R2" library="rcl" library_urn="urn:adsk.eagle:library:334" deviceset="R-EU_" device="0204/5" package3d_urn="urn:adsk.eagle:package:23488/1" value="100k"/>
 <part name="SUPPLY1" library="SparkFun-PowerSymbols" deviceset="VDD" device="" value="PA0"/>
+<part name="P+1" library="supply1" library_urn="urn:adsk.eagle:library:371" deviceset="V+" device=""/>
+<part name="P-1" library="supply1" library_urn="urn:adsk.eagle:library:371" deviceset="V-" device=""/>
 </parts>
 <sheets>
@@
 </plain>
 <instances>
-<instance part="VD1" gate="G$1" x="167.64" y="96.52" rot="R90">
+<instance part="VD1" gate="G$1" x="167.64" y="96.52" smashed="yes" rot="R90">
 <attribute name="NAME" x="165.735" y="94.742" size="1.778" layer="95" rot="R90"/>
 <attribute name="VALUE" x="171.069" y="94.742" size="1.778" layer="96" rot="R90"/>
 </instance>
-<instance part="D1" gate="1" x="172.72" y="66.04" rot="R90">
+<instance part="D1" gate="1" x="172.72" y="66.04" smashed="yes" rot="R90">
 <attribute name="NAME" x="172.2374" y="68.58" size="1.778" layer="95" rot="R90"/>
 <attribute name="VALUE" x="175.0314" y="68.58" size="1.778" layer="96" rot="R90"/>
 </instance>
-<instance part="VT2" gate="G$1" x="175.26" y="86.36" rot="MR180">
+<instance part="VT2" gate="G$1" x="175.26" y="86.36" smashed="yes" rot="MR180">
 <attribute name="VALUE" x="163.83" y="83.82" size="1.778" layer="96" rot="MR180"/>
 <attribute name="NAME" x="163.83" y="86.36" size="1.778" layer="95" rot="MR180"/>
 </instance>
-<instance part="IRON" gate="G$1" x="190.5" y="68.58">
+<instance part="IRON" gate="G$1" x="190.5" y="68.58" smashed="yes">
 <attribute name="NAME" x="184.15" y="74.295" size="1.778" layer="95"/>
 <attribute name="VALUE" x="184.15" y="63.5" size="1.778" layer="96"/>
 </instance>
-<instance part="GND9" gate="1" x="180.34" y="48.26">
+<instance part="GND9" gate="1" x="180.34" y="48.26" smashed="yes">
 <attribute name="VALUE" x="177.8" y="45.72" size="1.778" layer="96"/>
 </instance>
-<instance part="P+4" gate="1" x="180.34" y="129.54">
+<instance part="P+4" gate="1" x="180.34" y="129.54" smashed="yes">
 <attribute name="VALUE" x="177.8" y="124.46" size="1.778" layer="96" rot="R90"/>
 </instance>
-<instance part="GND12" gate="1" x="149.86" y="63.5">
+<instance part="GND12" gate="1" x="149.86" y="63.5" smashed="yes">
 <attribute name="VALUE" x="147.32" y="60.96" size="1.778" layer="96"/>
 </instance>
-<instance part="VT1" gate="G$1" x="147.32" y="83.82">
+<instance part="VT1" gate="G$1" x="147.32" y="83.82" smashed="yes">
 <attribute name="NAME" x="152.4" y="83.82" size="1.778" layer="95"/>
 <attribute name="VALUE" x="152.4" y="81.28" size="1.778" layer="96"/>
 </instance>
-<instance part="R10" gate="G$1" x="180.34" y="60.96" rot="R90">
+<instance part="R10" gate="G$1" x="180.34" y="60.96" smashed="yes" rot="R90">
 <attribute name="NAME" x="178.8414" y="57.15" size="1.778" layer="95" rot="R90"/>
 <attribute name="VALUE" x="183.642" y="57.15" size="1.778" layer="96" rot="R90"/>
 </instance>
-<instance part="R1" gate="G$1" x="134.62" y="83.82">
+<instance part="R1" gate="G$1" x="134.62" y="83.82" smashed="yes">
 <attribute name="NAME" x="130.81" y="85.3186" size="1.778" layer="95"/>
 <attribute name="VALUE" x="130.81" y="80.518" size="1.778" layer="96"/>
 </instance>
-<instance part="R3" gate="G$1" x="149.86" y="71.12" rot="R90">
+<instance part="R3" gate="G$1" x="149.86" y="71.12" smashed="yes" rot="R90">
 <attribute name="NAME" x="148.3614" y="67.31" size="1.778" layer="95" rot="R90"/>
 <attribute name="VALUE" x="153.162" y="67.31" size="1.778" layer="96" rot="R90"/>
 </instance>
-<instance part="R2" gate="G$1" x="160.02" y="104.14" rot="R90">
+<instance part="R2" gate="G$1" x="160.02" y="104.14" smashed="yes" rot="R90">
 <attribute name="NAME" x="158.5214" y="100.33" size="1.778" layer="95" rot="R90"/>
 <attribute name="VALUE" x="163.322" y="100.33" size="1.778" layer="96" rot="R90"/>
 </instance>
-<instance part="SUPPLY1" gate="VDD" x="127" y="83.82" rot="R90">
+<instance part="SUPPLY1" gate="VDD" x="127" y="83.82" smashed="yes" rot="R90">
 <attribute name="VALUE" x="121.666" y="83.82" size="1.778" layer="96" rot="R180" align="bottom-center"/>
+</instance>
+<instance part="P+1" gate="1" x="198.12" y="71.12" smashed="yes" rot="R270">
+<attribute name="VALUE" x="198.12" y="73.66" size="1.778" layer="96"/>
+</instance>
+<instance part="P-1" gate="1" x="198.12" y="68.58" smashed="yes" rot="R90">
+<attribute name="VALUE" x="198.12" y="66.04" size="1.778" layer="96"/>
 </instance>
 </instances>
@@
 </segment>
 </net>
-<net name="N$16" class="0">
-<segment>
-<pinref part="IRON" gate="G$1" pin="2"/>
-<wire x1="180.34" y1="71.12" x2="187.96" y2="71.12" width="0.1524" layer="91"/>
-<wire x1="187.96" y1="71.12" x2="187.96" y2="68.58" width="0.1524" layer="91"/>
-<pinref part="IRON" gate="G$1" pin="1"/>
-<junction x="187.96" y="71.12"/>
-<junction x="187.96" y="68.58"/>
-<wire x1="180.34" y1="68.58" x2="187.96" y2="68.58" width="0.1524" layer="91"/>
-<wire x1="180.34" y1="66.04" x2="180.34" y2="68.58" width="0.1524" layer="91"/>
-<pinref part="R10" gate="G$1" pin="2"/>
-<wire x1="180.34" y1="78.74" x2="172.72" y2="78.74" width="0.1524" layer="91"/>
-<pinref part="D1" gate="1" pin="C"/>
-<wire x1="172.72" y1="78.74" x2="172.72" y2="68.58" width="0.1524" layer="91"/>
-<pinref part="VT2" gate="G$1" pin="D"/>
-<wire x1="180.34" y1="78.74" x2="180.34" y2="83.82" width="0.1524" layer="91"/>
-<junction x="180.34" y="78.74"/>
-<wire x1="180.34" y1="71.12" x2="180.34" y2="78.74" width="0.1524" layer="91"/>
-</segment>
-</net>
 <net name="N$23" class="0">
 <segment>
@@
 </segment>
 </net>
+<net name="V+" class="0">
+<segment>
+<wire x1="180.34" y1="71.12" x2="187.96" y2="71.12" width="0.1524" layer="91"/>
+<pinref part="IRON" gate="G$1" pin="1"/>
+<wire x1="180.34" y1="78.74" x2="172.72" y2="78.74" width="0.1524" layer="91"/>
+<pinref part="D1" gate="1" pin="C"/>
+<wire x1="172.72" y1="78.74" x2="172.72" y2="68.58" width="0.1524" layer="91"/>
+<pinref part="VT2" gate="G$1" pin="D"/>
+<wire x1="180.34" y1="78.74" x2="180.34" y2="83.82" width="0.1524" layer="91"/>
+<junction x="180.34" y="78.74"/>
+<wire x1="180.34" y1="71.12" x2="180.34" y2="78.74" width="0.1524" layer="91"/>
+<pinref part="P+1" gate="1" pin="V+"/>
+<wire x1="195.58" y1="71.12" x2="187.96" y2="71.12" width="0.1524" layer="91"/>
+<junction x="187.96" y="71.12"/>
+</segment>
+</net>
+<net name="V-" class="0">
+<segment>
+<pinref part="IRON" gate="G$1" pin="2"/>
+<pinref part="R10" gate="G$1" pin="2"/>
+<wire x1="180.34" y1="66.04" x2="180.34" y2="68.58" width="0.1524" layer="91"/>
+<wire x1="180.34" y1="68.58" x2="187.96" y2="68.58" width="0.1524" layer="91"/>
+<pinref part="P-1" gate="1" pin="V-"/>
+<wire x1="195.58" y1="68.58" x2="187.96" y2="68.58" width="0.1524" layer="91"/>
+<junction x="187.96" y="68.58"/>
+</segment>
+</net>
