File: eagle/handle.sch (EAGLE design)
At the start: 3 parts

Commit message: Add files via upload
Connections:
- net GND renamed V-
- net VCC renamed V+
Changed lines of the file:
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@@
 <?xml version="1.0" encoding="utf-8"?>
 <!DOCTYPE eagle SYSTEM "eagle.dtd">
-<eagle version="9.2.0">
+<eagle version="9.6.1">
 <drawing>
 <settings>
@@
 <part name="TILT" library="sensor-signalquest" deviceset="SQ-SEN-200" device="" value=""/>
 <part name="PE" library="SparkFun-PowerSymbols" deviceset="GND2" device="" value="PE"/>
-<part name="GND2" library="SparkFun-PowerSymbols" deviceset="GND" device=""/>
-<part name="SUPPLY1" library="SparkFun-PowerSymbols" deviceset="VCC" device="" value="+24v"/>
+<part name="P-1" library="supply1" library_urn="urn:adsk.eagle:library:371" deviceset="V-" device=""/>
+<part name="P+1" library="supply1" library_urn="urn:adsk.eagle:library:371" deviceset="V+" device=""/>
 </parts>
 <sheets>
@@
 </plain>
 <instances>
-<instance part="IRON" gate="G$1" x="40.64" y="88.9" rot="R270">
+<instance part="IRON" gate="G$1" x="40.64" y="88.9" smashed="yes" rot="R270">
 <attribute name="VALUE" x="30.48" y="90.17" size="1.778" layer="96" rot="R270"/>
 <attribute name="NAME" x="38.862" y="92.71" size="1.778" layer="95"/>
 </instance>
-<instance part="R13" gate="G$1" x="50.8" y="68.58" rot="R90">
+<instance part="R13" gate="G$1" x="50.8" y="68.58" smashed="yes" rot="R90">
 <attribute name="NAME" x="46.99" y="66.04" size="1.778" layer="95" rot="R90"/>
 <attribute name="VALUE" x="54.61" y="63.5" size="1.778" layer="96" rot="R90"/>
 </instance>
-<instance part="TILT" gate="G$1" x="63.5" y="68.58">
+<instance part="TILT" gate="G$1" x="63.5" y="68.58" smashed="yes">
 <attribute name="NAME" x="68.58" y="71.12" size="1.778" layer="95"/>
 <attribute name="VALUE" x="68.58" y="63.5" size="1.778" layer="95"/>
 </instance>
-<instance part="PE" gate="G$1" x="40.64" y="73.66">
+<instance part="PE" gate="G$1" x="40.64" y="73.66" smashed="yes">
 <attribute name="VALUE" x="40.64" y="71.882" size="1.778" layer="96" align="top-center"/>
 </instance>
-<instance part="GND2" gate="1" x="35.56" y="53.34">
-<attribute name="VALUE" x="35.56" y="53.086" size="1.778" layer="96" align="top-center"/>
-</instance>
-<instance part="SUPPLY1" gate="G$1" x="33.02" y="78.74" rot="R90">
-<attribute name="VALUE" x="27.686" y="78.74" size="1.778" layer="96" align="bottom-center"/>
+<instance part="P-1" gate="1" x="35.56" y="53.34" smashed="yes">
+<attribute name="VALUE" x="38.1" y="53.34" size="1.778" layer="96"/>
+</instance>
+<instance part="P+1" gate="1" x="30.48" y="78.74" smashed="yes" rot="R90">
+<attribute name="VALUE" x="30.48" y="81.28" size="1.778" layer="96" rot="R180"/>
 </instance>
 </instances>
@@
 </busses>
 <nets>
-<net name="VCC" class="0">
-<segment>
-<pinref part="IRON" gate="G$1" pin="1"/>
-<wire x1="35.56" y1="81.28" x2="35.56" y2="78.74" width="0.1524" layer="91"/>
-<pinref part="SUPPLY1" gate="G$1" pin="VCC"/>
-<wire x1="35.56" y1="78.74" x2="33.02" y2="78.74" width="0.1524" layer="91"/>
-</segment>
-</net>
 <net name="3.3V" class="0">
 <segment>
@@
 </segment>
 </net>
-<net name="GND" class="0">
+<net name="N$2" class="0">
+<segment>
+<pinref part="IRON" gate="G$1" pin="4"/>
+<wire x1="43.18" y1="81.28" x2="43.18" y2="76.2" width="0.1524" layer="91"/>
+<pinref part="R13" gate="G$1" pin="1"/>
+<wire x1="43.18" y1="76.2" x2="50.8" y2="76.2" width="0.1524" layer="91"/>
+<wire x1="50.8" y1="76.2" x2="50.8" y2="73.66" width="0.1524" layer="91"/>
+</segment>
+</net>
+<net name="N$3" class="0">
+<segment>
+<pinref part="TILT" gate="G$1" pin="1"/>
+<wire x1="63.5" y1="76.2" x2="63.5" y2="78.74" width="0.1524" layer="91"/>
+<wire x1="63.5" y1="78.74" x2="45.72" y2="78.74" width="0.1524" layer="91"/>
+<pinref part="IRON" gate="G$1" pin="5"/>
+<wire x1="45.72" y1="78.74" x2="45.72" y2="81.28" width="0.1524" layer="91"/>
+</segment>
+</net>
+<net name="V-" class="0">
 <segment>
 <pinref part="IRON" gate="G$1" pin="2"/>
 <wire x1="38.1" y1="81.28" x2="38.1" y2="76.2" width="0.1524" layer="91"/>
 <wire x1="38.1" y1="76.2" x2="35.56" y2="76.2" width="0.1524" layer="91"/>
-<pinref part="GND2" gate="1" pin="GND"/>
 <wire x1="35.56" y1="76.2" x2="35.56" y2="58.42" width="0.1524" layer="91"/>
 <pinref part="TILT" gate="G$1" pin="2"/>
@@
 <wire x1="50.8" y1="63.5" x2="50.8" y2="58.42" width="0.1524" layer="91"/>
 <junction x="50.8" y="58.42"/>
-</segment>
-</net>
-<net name="N$2" class="0">
-<segment>
-<pinref part="IRON" gate="G$1" pin="4"/>
-<wire x1="43.18" y1="81.28" x2="43.18" y2="76.2" width="0.1524" layer="91"/>
-<pinref part="R13" gate="G$1" pin="1"/>
-<wire x1="43.18" y1="76.2" x2="50.8" y2="76.2" width="0.1524" layer="91"/>
-<wire x1="50.8" y1="76.2" x2="50.8" y2="73.66" width="0.1524" layer="91"/>
-</segment>
-</net>
-<net name="N$3" class="0">
-<segment>
-<pinref part="TILT" gate="G$1" pin="1"/>
-<wire x1="63.5" y1="76.2" x2="63.5" y2="78.74" width="0.1524" layer="91"/>
-<wire x1="63.5" y1="78.74" x2="45.72" y2="78.74" width="0.1524" layer="91"/>
-<pinref part="IRON" gate="G$1" pin="5"/>
-<wire x1="45.72" y1="78.74" x2="45.72" y2="81.28" width="0.1524" layer="91"/>
-</segment>
-</net>
+<pinref part="P-1" gate="1" pin="V-"/>
+</segment>
+</net>
+<net name="V+" class="0">
+<segment>
+<pinref part="IRON" gate="G$1" pin="1"/>
+<wire x1="35.56" y1="81.28" x2="35.56" y2="78.74" width="0.1524" layer="91"/>
+<wire x1="35.56" y1="78.74" x2="33.02" y2="78.74" width="0.1524" layer="91"/>
+<pinref part="P+1" gate="1" pin="V+"/>
+</segment>
+</net>
